Commit message: Port to ROS 2 Jazzy and Gazebo Harmonic
Same estimation code, robot behavior, scenario and parameters of the
ROS 1 version.

- ament_cmake package with the messages (UwbData, RobotData) and the
  Python modules; nodes ported to rclpy, parameters in config/params.yaml
- launch/sim.launch.py replaces init.launch, start_nodes.launch and
  gazebo_init.py: spawning from the csv files, static transforms of the
  anchors, ros_gz bridge, nodes of every robot in its namespace
- Robot with Gazebo Harmonic systems (diff drive, odometry publisher,
  camera sensor); world with a clean GUI without side panels; colors
  instead of the Gazebo Classic material scripts
- camera_rate launch argument to keep the simulation fast without a GPU
- Analysis scripts read ROS 1 and ROS 2 bags with rosbags; reference
  run recorded in MCAP in bagfiles/total_bag
- Docker image on osrf/ros:jazzy-desktop-full, colcon build in CI

File: urdf/unicycle.urdf.xacro (robot description, xacro)
@@ -1,4 +1,9 @@
 <?xml version="1.0"?>
 <robot name="unicycle" xmlns:xacro="http://ros.org/wiki/xacro">
+<!-- Name of the robot, used for the namespace of its Gazebo topics -->
+<xacro:arg name="robot_name" default="robot0" />
+<xacro:property name="robot_name" value="$(arg robot_name)" />
+<!-- Frame rate of the camera, it can be lowered when Gazebo renders without a GPU -->
+<xacro:arg name="camera_rate" default="30" />
 <!-- Defining the colors used in this robot -->
 <material name="Black">
@@ -13,4 +18,7 @@
 <material name="Blue">
 <color rgba="0.0 0.0 0.8 1.0"/>
+</material>
+<material name="Grey">
+<color rgba="0.5 0.5 0.5 1.0"/>
 </material>
 <!-- PROPERTY LIST -->
@@ -69,5 +77,4 @@
 </link>
 <gazebo reference="base_ground">
-    <turnGravityOff>false</turnGravityOff>
 </gazebo>
 <joint name="base_ground_joint" type="fixed">
@@ -92,5 +99,5 @@
             <mesh filename="package://dist_project/mesh/base.stl" scale="0.01 0.01 0.01" />
         </geometry>
-        <material name="White" />
+        <material name="Red" />
     </visual>
     <collision>
@@ -102,6 +109,4 @@
 </link>
 <gazebo reference="base_link">
-    <material>Gazebo/Red</material>
-    <turnGravityOff>false</turnGravityOff>
 </gazebo>
 <link name="caster_front_link">
@@ -133,8 +138,6 @@
 </joint>
 <gazebo reference="caster_front_link">
-    <turnGravityOff>false</turnGravityOff>
     <mu1 value="0.000001"/>
     <mu2 value="0.000001"/>
-    <material>Gazebo/Black</material>
 </gazebo>
 <link name="caster_back_link">
@@ -166,8 +169,6 @@
 </joint>
 <gazebo reference="caster_back_link">
-    <turnGravityOff>false</turnGravityOff>
     <mu1 value="0.000001"/>
     <mu2 value="0.000001"/>
-    <material>Gazebo/Black</material>
 </gazebo>
 <!-- RIGHT WHEEL DEFINITION -->
@@ -178,7 +179,5 @@
         <mesh filename="package://dist_project/mesh/wheel.stl" scale="0.001 0.001 0.001" />
     </geometry>
-    <material name="Red">
-        <color rgba="0.8 0.0 0.0 1.0"/>
-    </material>
+    <material name="Grey" />
     </visual>
     <collision>
@@ -203,6 +202,4 @@
     <kd  value="1.0" />
     <fdir1 value="1 0 0"/>
-    <material>Gazebo/Grey</material>
-    <turnGravityOff>false</turnGravityOff>
 </gazebo>
 <joint name="front_right_wheel_joint" type="continuous">
@@ -231,7 +228,5 @@
         <mesh filename="package://dist_project/mesh/wheel.stl" scale="0.001 0.001 0.001" />
     </geometry>
-    <material name="Red">
-        <color rgba="0.8 0.0 0.0 1.0"/>
-    </material>
+    <material name="Grey" />
     </visual>
     <collision>
@@ -256,6 +251,4 @@
     <kd  value="1.0" />
     <fdir1 value="1 0 0"/>
-    <material>Gazebo/Grey</material>
-    <turnGravityOff>false</turnGravityOff>
 </gazebo>
 <joint name="front_left_wheel_joint" type="continuous">
@@ -299,9 +292,10 @@
 </joint>
 <gazebo reference="camera_link">
-    <material>Gazebo/Blue</material>
     <sensor name="camera" type="camera">
         <pose> 0 0 0 0 0 0 </pose>
+        <always_on>true</always_on>
+        <topic>/${robot_name}/camera/image_raw</topic>
         <visualize>true</visualize>
-        <update_rate>30</update_rate>
+        <update_rate>$(arg camera_rate)</update_rate>
         <camera>
             <horizontal_fov>2</horizontal_fov>
@@ -321,8 +315,4 @@
             </noise>
         </camera>
-        <plugin name="camera_controller" filename="libgazebo_ros_camera.so">
-            <frame_name>camera_optical_link</frame_name>
-            <cameraName>camera</cameraName>
-        </plugin>
     </sensor>
 </gazebo>
@@ -342,37 +332,26 @@
 </joint>
 <gazebo reference="camera_tip_link">
-    <turnGravityOff>false</turnGravityOff>
-    <material>Gazebo/Blue</material>
 </gazebo>
 <!-- Gazebo Plugins -->
 <gazebo>
-    <plugin name="differential_drive_controller" filename="libgazebo_ros_diff_drive.so">
-        <legacyMode>true</legacyMode>
-        <rosDebugLevel>Debug</rosDebugLevel>
-        <publishWheelTF>true</publishWheelTF>
-        <publishWheelJointState>true</publishWheelJointState>
-        <alwaysOn>true</alwaysOn>
-        <updateRate>10.0</updateRate>
-        <leftJoint>front_left_wheel_joint</leftJoint>
-        <rightJoint>front_right_wheel_joint</rightJoint>
-        <wheelSeparation>${base_width}</wheelSeparation>
-        <wheelDiameter>${2*wheel_radius}</wheelDiameter>
-        <broadcastTF>1</broadcastTF>
-        <wheelTorque>30</wheelTorque>
-        <wheelAcceleration>1.8</wheelAcceleration>
-        <commandTopic>cmd_vel</commandTopic>
-        <odometryFrame>odom</odometryFrame>
-        <odometryTopic>odom</odometryTopic>
-        <robotBaseFrame>base_ground</robotBaseFrame>
-        <odometrySource>world</odometrySource>
-        <publishTf>1</publishTf>
-        <publishOdomTF>true</publishOdomTF>
+    <!-- Differential drive: velocity commands in and wheel odometry out -->
+    <plugin filename="gz-sim-diff-drive-system" name="gz::sim::systems::DiffDrive">
+        <left_joint>front_left_wheel_joint</left_joint>
+        <right_joint>front_right_wheel_joint</right_joint>
+        <wheel_separation>${base_width}</wheel_separation>
+        <wheel_radius>${wheel_radius}</wheel_radius>
+        <topic>/${robot_name}/cmd_vel</topic>
+        <odom_topic>/${robot_name}/odom</odom_topic>
+        <odom_publish_frequency>10</odom_publish_frequency>
+        <frame_id>${robot_name}/odom</frame_id>
+        <child_frame_id>${robot_name}/base_ground</child_frame_id>
     </plugin>
-    <plugin name="p3d_base_controller" filename="libgazebo_ros_p3d.so">
-        <alwaysOn>true</alwaysOn>
-        <updateRate>10</updateRate>
-        <bodyName>base_link</bodyName>
-        <topicName>ground_truth/state</topicName>
-        <frameName>world</frameName>
+    <!-- Ground truth pose of the robot in the world frame -->
+    <plugin filename="gz-sim-odometry-publisher-system" name="gz::sim::systems::OdometryPublisher">
+        <odom_frame>world</odom_frame>
+        <robot_base_frame>${robot_name}/base_ground</robot_base_frame>
+        <odom_topic>/${robot_name}/ground_truth/state</odom_topic>
+        <odom_publish_frequency>10</odom_publish_frequency>
+        <dimensions>3</dimensions>
     </plugin>
 </gazebo>

Commit message: Faster simulation and camera fields of view in Gazebo
Gazebo publishes the clock at every physics step and every node read it,
so the nodes now get a 100 Hz clock through topic_tools throttle. The
fields of view of the robot cameras are drawn in the Gazebo view, hidden
to the cameras themselves.

File: urdf/unicycle.urdf.xacro (robot description, xacro)
@@ -300,4 +300,6 @@
         <camera>
             <horizontal_fov>2</horizontal_fov>
+            <!-- The camera doesn't see the field of view drawn below -->
+            <visibility_mask>1</visibility_mask>
             <image>
                 <format>R8G8B8</format>
@@ -316,4 +318,31 @@
         </camera>
     </sensor>
+</gazebo>
+<!-- Field of view of the camera, drawn in Gazebo as Gazebo Classic did with visualize -->
+<link name="camera_fov_link">
+    <visual>
+        <origin xyz="0 0 0" rpy="0 0 0" />
+        <geometry>
+            <mesh filename="package://dist_project/mesh/camera_fov.stl" />
+        </geometry>
+    </visual>
+</link>
+<joint name="camera_fov_joint" type="fixed">
+    <parent link="camera_link" />
+    <child link="camera_fov_link" />
+    <origin xyz="0 0 0" rpy="0 0 0" />
+</joint>
+<gazebo reference="camera_fov_link">
+    <!-- Only the Gazebo view shows it, the cameras have visibility_mask 1 -->
+    <visual>
+        <cast_shadows>false</cast_shadows>
+        <transparency>0.8</transparency>
+        <visibility_flags>2</visibility_flags>
+        <material>
+            <ambient>0.3 0.6 1 1</ambient>
+            <diffuse>0.3 0.6 1 1</diffuse>
+            <emissive>0.1 0.2 0.35 1</emissive>
+        </material>
+    </visual>
 </gazebo>
 <link name="camera_tip_link">
